Commit message: init

File: urdf/maze_solver.urdf (robot description, URDF)
Before this commit: robot maze_solver, 11 links, 10 joints
Links:
- removed link sensor_b
- added link sensor_l, mass 0.000400000000000001; collision mesh filename=package://maze_solver/meshes/sensor_l.STL; visual mesh filename=package://maze_solver/meshes/sensor_l.STL
- link arm_base: mass 0.0449400000000001 -> 0.0449400000000003
- link arm_top: mass 0.0449400000000001 -> 0.0449399999999996
- link camera: mass 0.0641999999999999 -> 0.0642
- link sensor_f: mass 0.000399999999999999 -> 0.0004
- link sensor_r: mass 0.000399999999999999 -> 0.000400000000000001
- link wheel_l: mass 0.0282743338823081 -> 0.0282743338823082
Joints:
- removed joint sensor_b_joint
- added joint sensor_l_joint: type fixed, parent base_link, child sensor_l, origin xyz=0.19 0.00167825063166787 0.261284591199386 rpy=3.14159265358979 0 -1.5707963267949, axis 0 0 0
- joint arm_base_joint: limit lower=0 upper=1.5708 effort=0 velocity=0 -> lower=-0.219374105739371 upper=1.35142222105552 effort=0 velocity=0; origin xyz=0.46201 -0.28163 0.35327 rpy=1.5708 0 0 -> xyz=0.189999999999998 0.0250000000000001 0.265000000000002 rpy=1.5707963267949 0.219374105739364 0
- joint arm_top_joint: limit lower=0 upper=3.1416 effort=0 velocity=0 -> lower=-0.514515495694073 upper=2.62707715789572 effort=0 velocity=0; origin xyz=-0.38 0.01 0 rpy=0 0 0 -> xyz=-0.379999999999998 0.00999999999999857 0 rpy=0 0 0.514515495694071
- joint camera: origin xyz=0.35232 0.01 0.028889 rpy=1.5708 1.5708 1.5708 -> xyz=0.352324176953221 0.0100000000000041 0.0288889997713121 rpy=0.590282779909414 1.5707963267949 0
- joint caster_b_joint: axis 0 0 0 -> 0 1 0; origin xyz=0.27201 -0.39288 0.069514 rpy=1.5708 0 0 -> xyz=0 0.08625 0 rpy=1.5707963267949 0 0; type fixed -> continuous
- joint caster_f_joint: origin xyz=0.27201 -0.22038 0.068372 rpy=1.5708 0 0 -> xyz=0 -0.08625 0 rpy=1.5707963267949 0 0.599335912665456; type fixed -> continuous
- joint sensor_f_joint: origin xyz=0.270394416349372 -0.331632232073919 0.344987084647221 rpy=3.14159265358979 0 0 -> xyz=-0.00161067072073706 -0.0249999999999999 0.256715408800614 rpy=3.14159265358979 0 0
- joint sensor_r_joint: origin xyz=0.077005 -0.30495 0.35156 rpy=3.1416 0 -1.5708 -> xyz=-0.195 0.00167825063166793 0.263284591199386 rpy=3.14159265358979 0 -1.5707963267949
- joint wheel_l_joint: axis 1 0 0 -> 0 0 1; origin xyz=0.082005 -0.26955 0.098272 rpy=-1.5708 0 -1.5708 -> xyz=0.19 0 0.01 rpy=1.5707963267949 0.885460579278242 1.5707963267949; type revolute -> continuous
- joint wheel_r_joint: axis 0.63293 0.77421 0 -> 0 0 1; origin xyz=0.46201 -0.25734 0.098272 rpy=1.5708 0.88546 1.5708 -> xyz=-0.19 0 0.01 rpy=1.5707963267949 1.30809386854526 -1.5707963267949; type revolute -> continuous

Commit message: Added Differential Drive

File: urdf/maze_solver.urdf (robot description, URDF)
Before this commit: robot maze_solver, 11 links, 10 joints
Joints:
- joint arm_base_joint: limit lower=-0.219374105739371 upper=1.35142222105552 effort=0 velocity=0 -> lower=-0.219374105739371 upper=0.21 effort=0 velocity=0
- joint wheel_l_joint: axis 0 0 1 -> 0 0 -1

Commit message: Fixed Bug

File: urdf/maze_solver.urdf (robot description, URDF)
Before this commit: robot maze_solver, 11 links, 10 joints
Links:
- link caster_b: geometry collision sphere radius=0.02; visual mesh filename=package://maze_solver/meshes/caster_b.STL
- link caster_f: geometry collision sphere radius=0.02; visual mesh filename=package://maze_solver/meshes/caster_f.STL
Joints:
- joint caster_b_joint: axis 0 1 0 -> (none)
- joint caster_f_joint: axis 0 1 0 -> (none)

Commit message: IR Sensor

File: urdf/maze_solver.urdf (robot description, URDF)
Before this commit: robot maze_solver, 11 links, 10 joints
Joints:
- joint sensor_f_joint: origin xyz=-0.00161067072073706 -0.0249999999999999 0.256715408800614 rpy=3.14159265358979 0 0 -> xyz=-0.00161067072073706 -0.0249999999999999 0.256715408800614 rpy=3.14159265358979 0 -1.57
- joint sensor_l_joint: origin xyz=0.19 0.00167825063166787 0.261284591199386 rpy=3.14159265358979 0 -1.5707963267949 -> xyz=0.19 0.00167825063166787 0.261284591199386 rpy=3.14159265358979 0 0
- joint sensor_r_joint: origin xyz=-0.195 0.00167825063166793 0.263284591199386 rpy=3.14159265358979 0 -1.5707963267949 -> xyz=-0.195 0.00167825063166793 0.263284591199386 rpy=3.14159265358979 0 -3.14
- joint wheel_l_joint: axis 0 0 -1 -> 0 0 1
- joint wheel_r_joint: axis 0 0 1 -> 0 0 -1

Commit message: Maze Solved!

File: urdf/maze_solver.urdf (robot description, URDF)
Before this commit: robot maze_solver, 11 links, 10 joints
Joints:
- joint arm_base_joint: type revolute -> fixed
- joint arm_top_joint: type revolute -> fixed

Commit message: Small Changes

File: urdf/maze_solver.urdf (robot description, URDF)
Before this commit: robot maze_solver, 11 links, 10 joints
Joints:
- joint arm_base_joint: limit lower=-0.219374105739371 upper=0.21 effort=0 velocity=0 -> lower=-0.40 upper=-0.40 effort=0 velocity=0; type fixed -> revolute
- joint arm_top_joint: limit lower=-0.514515495694073 upper=2.62707715789572 effort=0 velocity=0 -> lower=1.63 upper=1.63 effort=0 velocity=0; type fixed -> revolute
- joint camera: axis 0 0 0 -> (none); origin xyz=0.352324176953221 0.0100000000000041 0.0288889997713121 rpy=0.590282779909414 1.5707963267949 0 -> xyz=0.352324176953221 0.0100000000000041 0.0288889997713121 rpy=0 0 1.57

Commit message: Final Version!

File: urdf/maze_solver.urdf (robot description, URDF)
Before this commit: robot maze_solver, 11 links, 10 joints
Joints:
- joint camera: origin xyz=0.352324176953221 0.0100000000000041 0.0288889997713121 rpy=0 0 1.57 -> xyz=0.352324176953221 0.0100000000000041 0.0288889997713121 rpy=0 -1.57 1.57
